File: Hardware/SparkFun_Qwiic_Fingerprint_Sensor_FPC2534.kicad_pcb (KiCad board)
At the start: 4 copper layers, 25.4 x 25.4 mm, 78 parts, among them J1 Qwiic_RA, J2 Qwiic_RA, J4 USB_C_Receptacle, J5 Conn_01x06, J7 Conn_01x06, U1 FPC2354, U2 RT9080-3.3

Commit message: Add I2C pull ups and jumper. Adjust silk.
Parts:
- removed kibuzzard-65A8A8B4: G***, kibuzzard-65A8A8B4
- removed kibuzzard-68825977: G***, kibuzzard-68825977
- removed kibuzzard-6882597D: G***, kibuzzard-6882597D
- removed kibuzzard-68825988 (x2): G***, kibuzzard-68825988
- removed kibuzzard-68825B75: G***, kibuzzard-68825B75
- removed kibuzzard-68825B8B: G***, kibuzzard-68825B8B
- removed kibuzzard-68825BEF: G***, kibuzzard-68825BEF
- removed kibuzzard-68825BF8: G***, kibuzzard-68825BF8
- removed kibuzzard-68825C08: G***, kibuzzard-68825C08
- removed kibuzzard-68825C0D: G***, kibuzzard-68825C0D
- removed kibuzzard-68825C35: G***, kibuzzard-68825C35
- removed kibuzzard-68825C4C: G***, kibuzzard-68825C4C
- removed kibuzzard-68825C7A: G***, kibuzzard-68825C7A
- removed kibuzzard-68825C89: G***, kibuzzard-68825C89
- removed kibuzzard-68825CB4 (x2): G***, kibuzzard-68825CB4
- removed kibuzzard-68825CBE (x2): G***, kibuzzard-68825CBE
- removed kibuzzard-68825CEF (x2): G***, kibuzzard-68825CEF
- removed kibuzzard-68825CF7 (x2): G***, kibuzzard-68825CF7
- removed kibuzzard-68825CFB (x2): G***, kibuzzard-68825CFB
- removed kibuzzard-68825D00 (x2): G***, kibuzzard-68825D00
- removed kibuzzard-68825D85: G***, kibuzzard-68825D85
- removed kibuzzard-68825E15: G***, kibuzzard-68825E15
- removed kibuzzard-68825E2B: G***, kibuzzard-68825E2B
- removed kibuzzard-68825E3F: G***, kibuzzard-68825E3F
- removed kibuzzard-6882609D: G***, kibuzzard-6882609D
- removed kibuzzard-688260A2: G***, kibuzzard-688260A2
- removed kibuzzard-6886EE7C: G***, kibuzzard-6886EE7C
- removed kibuzzard-6886EE9A: G***, kibuzzard-6886EE9A
- removed kibuzzard-6886F4FB: G***, kibuzzard-6886F4FB
- added JP4: I2C, SparkFun-Jumper:Jumper_3_NC-2_Trace, B.Cu at (127.1, 98.1)
- added R11: 2.2k, SparkFun-Resistor:R_0603_1608Metric, F.Cu at (129.6, 101.0)
- added R12: 2.2k, SparkFun-Resistor:R_0603_1608Metric, F.Cu at (129.6, 98.1)
- added kibuzzard-68A62B00: G***, kibuzzard-68A62B00, B.Cu at (127.1, 100.0)
- added kibuzzard-68B210FC: G***, kibuzzard-68B210FC, F.Cu at (127.4, 110.2)
- added kibuzzard-68B21103: G***, kibuzzard-68B21103, F.Cu at (133.4, 108.3)
- added kibuzzard-68B2110A: G***, kibuzzard-68B2110A, F.Cu at (136.0, 108.3)
- added kibuzzard-68B21113: G***, kibuzzard-68B21113, F.Cu at (138.5, 108.3)
- added kibuzzard-68B21123: G***, kibuzzard-68B21123, F.Cu at (141.0, 108.3)
- added kibuzzard-68B21136: G***, kibuzzard-68B21136, F.Cu at (144.5, 110.2)
- added kibuzzard-68B21145: G***, kibuzzard-68B21145, F.Cu at (136.0, 102.2)
- added kibuzzard-68B21150: G***, kibuzzard-68B21150, F.Cu at (136.0, 100.6)
- added kibuzzard-68B21159: G***, kibuzzard-68B21159, F.Cu at (128.0, 102.6)
- added kibuzzard-68B21162: G***, kibuzzard-68B21162, F.Cu at (131.2, 94.9)
- added kibuzzard-68B21169: G***, kibuzzard-68B21169, F.Cu at (140.9, 94.9)
- added kibuzzard-68B21179: G***, kibuzzard-68B21179, B.Cu at (145.2, 96.5)
- added kibuzzard-68B21181: G***, kibuzzard-68B21181, B.Cu at (145.2, 98.1)
- added kibuzzard-68B2118A: G***, kibuzzard-68B2118A, B.Cu at (145.2, 99.4)
- added kibuzzard-68B21196: G***, kibuzzard-68B21196, B.Cu at (145.6, 104.8)
- added kibuzzard-68B2119E: G***, kibuzzard-68B2119E, B.Cu at (144.5, 110.2)
- added kibuzzard-68B211A8: G***, kibuzzard-68B211A8, B.Cu at (138.5, 108.3)
- added kibuzzard-68B211AF: G***, kibuzzard-68B211AF, B.Cu at (136.0, 108.3)
- added kibuzzard-68B211BC: G***, kibuzzard-68B211BC, B.Cu at (133.4, 108.3)
- added kibuzzard-68B211C4: G***, kibuzzard-68B211C4, B.Cu at (130.9, 108.3)
- added kibuzzard-68B211CC: G***, kibuzzard-68B211CC, B.Cu at (127.4, 110.2)
- added kibuzzard-68B21259: G***, kibuzzard-68B21259, B.Cu at (128.3, 92.4)
- added kibuzzard-68B21262: G***, kibuzzard-68B21262, B.Cu at (143.4, 92.4)
- added kibuzzard-68B2127B: G***, kibuzzard-68B2127B, B.Cu at (139.8, 104.6)
- added kibuzzard-68B21280: G***, kibuzzard-68B21280, B.Cu at (142.3, 104.6)
- added kibuzzard-68B21288: G***, kibuzzard-68B21288, B.Cu at (137.2, 104.9)
- added kibuzzard-68B21290: G***, kibuzzard-68B21290, B.Cu at (132.2, 104.9)
- added kibuzzard-68B21298: G***, kibuzzard-68B21298, B.Cu at (129.6, 104.8)
- added kibuzzard-68B212A1: G***, kibuzzard-68B212A1, B.Cu at (125.2, 102.6)
- added kibuzzard-68B212B8: G***, kibuzzard-68B212B8, F.Cu at (142.3, 104.5)
- added kibuzzard-68B212BF: G***, kibuzzard-68B212BF, F.Cu at (139.8, 104.5)
- added kibuzzard-68B212C8: G***, kibuzzard-68B212C8, F.Cu at (137.2, 104.8)
- added kibuzzard-68B212CF: G***, kibuzzard-68B212CF, F.Cu at (134.7, 105.1)
- added kibuzzard-68B212D5: G***, kibuzzard-68B212D5, F.Cu at (132.2, 104.9)
- added kibuzzard-68B212DD: G***, kibuzzard-68B212DD, F.Cu at (129.6, 104.8)
- added kibuzzard-68B21331: G***, kibuzzard-68B21331, F.Cu at (136.0, 92.7)
- moved C5 0.32 mm to (131.2, 98.1)
Routing:
- net SDA: track 29.1 -> 40.1 mm, vias 3 -> 2
- net 3.3V: track 67.3 -> 77.0 mm, vias 5 -> 6
- net Net-(JP4-C): track 0.00 -> 4.69 mm, vias 0 -> 1
- net Net-(JP4-A): track 0.00 -> 4.24 mm, vias 0 -> 1
- net GND: track 11.4 -> 13.7 mm
- net SCL: track 34.9 -> 36.8 mm

Commit message: Post design review.
Parts:
- removed ST1, ST2, ST3, ST4: Standoff, SparkFun-Hardware:Standoff
- removed TP3, TP4: TestPoint_0.75mm, SparkFun-Connector:TestPoint-0.75mm
- removed kibuzzard-68825C3B: G***, kibuzzard-68825C3B
- removed kibuzzard-68B210FC: G***, kibuzzard-68B210FC
- removed kibuzzard-68B21136: G***, kibuzzard-68B21136
- removed kibuzzard-68B2119E: G***, kibuzzard-68B2119E
- removed kibuzzard-68B211CC: G***, kibuzzard-68B211CC
- removed kibuzzard-68B21288: G***, kibuzzard-68B21288
- removed kibuzzard-68B21290: G***, kibuzzard-68B21290
- removed kibuzzard-68B21298: G***, kibuzzard-68B21298
- removed kibuzzard-68B212B8: G***, kibuzzard-68B212B8
- removed kibuzzard-68B212BF: G***, kibuzzard-68B212BF
- removed kibuzzard-68B212C8: G***, kibuzzard-68B212C8
- removed kibuzzard-68B212CF: G***, kibuzzard-68B212CF
- removed kibuzzard-68B212D5: G***, kibuzzard-68B212D5
- removed kibuzzard-68B212DD: G***, kibuzzard-68B212DD
- added J3: Conn_01x01, SparkFun-Connector:1x01, F.Cu at (142.3, 86.7)
- added J6: Conn_01x01, SparkFun-Connector:1x01, F.Cu at (129.6, 86.7)
- added JP5: BZL, SparkFun-Jumper:Jumper_2_NC_Trace, F.Cu at (144.2, 92.7)
- added ST5: Standoff, SparkFun-Hardware:Standoff_Connected, F.Cu at (125.8, 87.9)
- added ST6: Standoff, SparkFun-Hardware:Standoff_Connected, F.Cu at (146.1, 87.9)
- added ST7: Standoff, SparkFun-Hardware:Standoff_Connected, F.Cu at (146.1, 108.3)
- added ST8: Standoff, SparkFun-Hardware:Standoff_Connected, F.Cu at (125.8, 108.3)
- added kibuzzard-68B21162: G***, kibuzzard-68B21162, B.Cu at (129.6, 88.9)
- added kibuzzard-68B21169: G***, kibuzzard-68B21169, B.Cu at (142.3, 88.9)
- added kibuzzard-68BB5A49: G***, kibuzzard-68BB5A49, F.Cu at (140.7, 94.9)
- added kibuzzard-68BB5B69: G***, kibuzzard-68BB5B69, F.Cu at (129.6, 104.8)
- added kibuzzard-68BB5B72: G***, kibuzzard-68BB5B72, F.Cu at (132.2, 105.1)
- added kibuzzard-68BB5B7A: G***, kibuzzard-68BB5B7A, F.Cu at (134.7, 105.1)
- added kibuzzard-68BB5B86: G***, kibuzzard-68BB5B86, F.Cu at (139.8, 104.5)
- added kibuzzard-68BB5B8B: G***, kibuzzard-68BB5B8B, F.Cu at (142.3, 104.5)
- added kibuzzard-68BB5BA4: G***, kibuzzard-68BB5BA4, B.Cu at (134.7, 105.1)
- added kibuzzard-68BB5BAA: G***, kibuzzard-68BB5BAA, B.Cu at (132.2, 105.1)
- added kibuzzard-68BB5BB0: G***, kibuzzard-68BB5BB0, B.Cu at (129.6, 104.6)
- added kibuzzard-68BB5BE0: G***, kibuzzard-68BB5BE0, F.Cu at (137.2, 104.9)
- added kibuzzard-68BB5BFB: G***, kibuzzard-68BB5BFB, B.Cu at (137.2, 104.7)
- added kibuzzard-68C08F5C: G***, kibuzzard-68C08F5C, F.Cu at (130.9, 108.3)
- added kibuzzard-68C08F6E: G***, kibuzzard-68C08F6E, F.Cu at (143.3, 108.3)
- added kibuzzard-68C08F6E: G***, kibuzzard-68C08F6E, B.Cu at (141.0, 108.3)
- added kibuzzard-68C08FA6: G***, kibuzzard-68C08FA6, B.Cu at (128.7, 108.3)
- added kibuzzard-68C0923F: G***, kibuzzard-68C0923F, F.Cu at (141.4, 92.7)
- moved kibuzzard-68B21162 6.43 mm to (129.0, 88.9), turned to 90 degrees
- moved kibuzzard-68B21169 6.38 mm to (143.0, 88.9), turned to 90 degrees
- moved R2 0.95 mm to (130.3, 89.5)
- moved R4 0.95 mm to (141.7, 89.5)
- moved kibuzzard-68B2127B 0.16 mm to (139.8, 104.5)
- moved kibuzzard-68B21280 0.16 mm to (142.3, 104.5)
Connections:
- U1 pad A1: GND -> EGND
- U1 pad A8: GND -> EGND
- U1 pad H1: GND -> EGND
- U1 pad H8: GND -> EGND
Routing:
- net EGND: track 0.00 -> 13.3 mm, vias 0 -> 4
- net SDA: track 40.1 -> 51.5 mm, vias 2 -> 3
- net GND: track 13.7 -> 22.6 mm, vias 14 -> 22
- net SCL: track 36.8 -> 45.6 mm
- net 3.3V: track 77.0 -> 78.2 mm
- net ~{CS}: track 17.7 -> 18.7 mm
- net Net-(J4-CC2): track 7.04 -> 6.09 mm
- net DP: track 17.5 -> 16.7 mm
- net CFG1: track 15.2 -> 14.4 mm
- net DM: track 16.7 -> 16.1 mm
- added copper zone on In2.Cu, net EGND
- removed copper zone on In2.Cu, net GND
Other:
- board text added: "v11"
- board text removed: "v10"
